File: electronics/domcape/domcape.sch (KiCad schematic (older format))
At the start: 49 parts, among them P8 BeagleBone_Black_Header, SH-4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, P9 BeagleBone_Black_Header, SH-4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, Q1 SQ2348ES, Q2 SQ2303ES, U100 TLP291-4, U101 TLP291-4, U102 TLP291-4, U103 TLP291-4, U104 TLP291-4, U105 TLP291-4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

Commit message: add notes, and minor changes
Parts:
- R1: value 1000G -> placemaker
Changed lines of the file:
@@
 P 9450 9900
 F 0 "R1" V 9530 9900 50  0000 C CNN
-F 1 "1000G" V 9450 9900 50  0000 C CNN
+F 1 "placemaker" V 9450 9900 50  0000 C CNN
 F 2 "Resistors_SMD:R_0402" V 9380 9900 50  0000 C CNN
 F 3 "" H 9450 9900 50  0000 C CNN
